File: Atlas.kicad_sch (KiCad schematic)
At the start: 51 parts, among them J101 BATT, J102 GND, J103 A, J104 B, J105 C, J106 Conn_01x05, U101 INA186A2QDBVRQ1, U102 LMR51420YDDCR, U103 TLV76733DRVR

Commit message: deleted voltage sensing circuit, cleaned up wires organized redid reference desginator numbers ready for pcb design
Parts:
- removed J103: A, TestPoint:TestPoint_Pad_4.0x4.0mm, symbol Connector_Generic:Conn_01x01
- removed J104: B, TestPoint:TestPoint_Pad_4.0x4.0mm, symbol Connector_Generic:Conn_01x01
- removed J105: C, TestPoint:TestPoint_Pad_4.0x4.0mm, symbol Connector_Generic:Conn_01x01
- removed J106: Conn_01x05, symbol Connector_Generic:Conn_01x05
- removed TP105, TP106: TestPoint, symbol Connector:TestPoint
- added J104: Conn_01x08_MountingPin, Connector_JST:JST_SH_SM08B-SRSS-TB_1x08-1MP_P1.00mm_Horizontal, symbol Connector_Generic_MountingPin:Conn_01x08_MountingPin
- U101: value INA186A2QDBVRQ1 -> INA186A2
Connections:
- net +BATT: now also J104.1 (Pin_1)
- net CURRENT: now also J104.3 (Pin_3)
- net GND: now also J104.2 (Pin_2), J104.MP (MountPin)
- net TELEMETRY: now also J104.4 (Pin_4)
- new net M1: J104.5 (Pin_5)
- new net M2: J104.6 (Pin_6)
- new net M3: J104.7 (Pin_7)
- new net M4: J104.8 (Pin_8)
Other:
- sheet Motor_1 ports: added TELEMETRY; removed OUTPUT
- sheet Motor_2 ports: added SIGNAL_INPUT, TELEMETRY; removed none
- sheet Motor_3 ports: added SIGNAL_INPUT, TELEMETRY; removed none
- sheet Motor_4 ports: added SIGNAL_INPUT, TELEMETRY; removed none
- note added: "TVS DIODES"
- note removed: "MOTOR PADS"
- moved on the sheet: C101, C102, D101, D102, D107, D108, H101, H102, H103, H104, J101, J102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
